File: KiCad/v0.3/RP2040-Decoder.kicad_sch (KiCad schematic)
At the start: 57 parts, among them J1 T0, J10 2, J11 3, J12 4, J13 5, J14 +V, J15 M_OUT_B, J16 M_OUT_A, J17 GND, J18 SWCLK, J19 SWDIO, J2 T1, J20 RUN, J3 0, J4 1, J5 2, J6 3, J7 +3V3, J8 0, J9 1, Q1 T2N7002BK, Q2 T2N7002BK, Q3 T2N7002BK, Q4 T2N7002BK, Q5 T2N7002BK, U1 PJ75AL33SA, U2 BDR6133, U3 W25Q64JVSSIQ, U4 RP2040, Y1 X322512MSB4SI

Commit message: changes
Parts:
- removed C7: 100n, Capacitor_SMD:C_0201_0603Metric, symbol Device:C
- C1, C14, C2, C6: footprint RP2040-Decoder_Additional_Footprints:C_0603_1608Metric -> Capacitor_SMD:C_0402_1005Metric
- C17: footprint RP2040-Decoder_Additional_Footprints:C_0603_1608Metric -> Capacitor_SMD:C_0201_0603Metric
- C5: footprint Capacitor_SMD:C_0201_0603Metric -> Capacitor_SMD:C_0402_1005Metric
- J1, J10, J11, J12, J13, J14, J15, J16, J17, J18, J19, J2, J20, J3, J4, J5, J6, J7, J8, J9: footprint TestPoint:TestPoint_Pad_D2.0mm -> TestPoint:TestPoint_Pad_D1.5mm
- R2, R4, R5, R6, R7, R8: footprint RP2040-Decoder_Additional_Footprints:R_0603_1608Metric -> Resistor_SMD:R_0201_0603Metric
- R3: footprint RP2040-Decoder_Additional_Footprints:R_0603_1608Metric -> Capacitor_SMD:C_0402_1005Metric
- U4: footprint RP2040-Decoder_Additional_Footprints:QFN-56-1EP_7x7mm_P0.4mm_EP3.2x3.2mm -> User:QFN-56-1EP_7x7mm_P0.4mm_EP3.2x3.2mm_BigThermalVias
